File: PCB/LPT_Capture.kicad_pcb (KiCad board)
At the start: 2 copper layers, 36 x 20.8 mm, 16 parts, among them J1 USB3155-30-A, J2 DB25M, U1 FT245RL

Commit message: USBC
Parts:
- added R2: 5k1, 000_LOCAL:R_0805, F.Cu at (149.5, 100.5)
- added R3: 5k1, 000_LOCAL:R_0805, F.Cu at (147.4, 100.5)
- J1: value USB3155-30-A -> GSB1C4621DS2HR; footprint 000_LOCAL:GCT_USB3155-XX-X -> 000_LOCAL:USBC_16pin_mid_mount
- J2: value DB25M -> DB25P064TXLF
- N1: value DB25_backshell -> 956-025-010R031
- moved C3 5.52 mm to (151.5, 100.5), turned to 90 degrees
- moved C4 4.09 mm to (143.5, 100.5), turned to -90 degrees
- moved REF** 3.95 mm to (166.1, 111.1)
- moved C2 2.82 mm to (153.4, 100.5), turned to 90 degrees
- moved FB1 2.37 mm to (145.4, 100.5), turned to -90 degrees
- moved J1 1.90 mm to (150.0, 110.9)
- moved C1 0.78 mm to (155.3, 100.5), turned to 90 degrees
- moved REF** 0.61 mm to (135.0, 96.0)
- moved REF** 0.56 mm to (135.0, 110.0)
- renumbered C3 to C2, C2 to C3
Routing:
- net VBUS: track 5.43 -> 24.6 mm, vias 0 -> 6
- net Net-(J1-CC2): track 0.00 -> 5.79 mm
- net Net-(J1-CC1): track 0.00 -> 5.18 mm
- net VCC: track 37.3 -> 41.4 mm, vias 6 -> 8
- net /~{TXE}: track 22.5 -> 20.7 mm
- net /USB+: track 15.2 -> 13.6 mm, vias 0 -> 3
- net /USB-: track 15.1 -> 14.7 mm, vias 0 -> 2
- net GND: vias 18 -> 35
Other:
- board size 36 x 20.8 mm -> 36 x 22.8 mm
