File: PCB/LPT_Capture_DB25_MicroUSB_FANCY.kicad_sch (KiCad schematic)
At the start: 13 parts, among them J1 USB3155-30-A, J2 DB25P064TXLF, U1 FT245RL

Commit message: pull db25_microusb_fancy into main
Parts:
- removed C3: 0.1u, 000_LOCAL:C_0805, symbol 000_LOCAL:C_Small
- added C2: 0.1u, 000_LOCAL:C_0805, symbol 000_LOCAL:C_Small
- added LED1: ONLINE, 000_LOCAL:LED_0805, symbol 000_LOCAL:LED
- added LED2: SELECT, 000_LOCAL:LED_0805, symbol 000_LOCAL:LED
- added Q1, Q2: SL2301S, 000_LOCAL:SOT-23, symbol 000_LOCAL:PMOS_GSD
- added R2, R3, R4, R5: 10k, 000_LOCAL:R_0805, symbol 000_LOCAL:R_Small
- J1: footprint USB3155-xx-x -> 000_LOCAL:USB3155-xx-x; symbol 000_LOCAL:USB3155-xx-x -> 000_LOCAL:USB3155-XX-X_REVA; MANUFACTURER GCT -> (none)
- R1: value 47k -> 10k; MPN RC0805JR-0747KL -> RC0805JR-0710KL
- U1: footprint 000_LOCAL:SSOP-28 -> 000_LOCAL:SSOP-28_5.3x10.2mm_P0.65mm
- renumbered C2 to C3
Connections:
- net 3v3: now also C1.2; no longer C1.1
- net D2: now also RA2.4 (R4.1); no longer RA3.1 (R1.1)
- net D3: now also RA2.3 (R3.1); no longer RA2.4 (R4.1)
- net D4: now also RA2.2 (R2.1); no longer RA2.3 (R3.1)
- net D5: now also RA2.1 (R1.1); no longer RA2.2 (R2.1)
- net D6: now also RA1.4 (R4.1); no longer RA2.1 (R1.1)
- net D7: now also RA1.3 (R3.1); no longer RA1.4 (R4.1)
- net GND: now also C1.1, C2.2, R4.2, R5.2; no longer C1.2
- net ONLINE: now also RA1.1 (R1.1), LED1.2 (A), LED2.2 (A), Q1.3 (D); no longer J2.13, RA1.8 (R1.2)
- net VCC: now also C2.1, Q1.2 (S), R2.2, R3.2; no longer RA1.1 (R1.1), U1.19 (~{RESET})
- net ~{RESET}: now also RA3.1 (R1.1), U1.19 (~{RESET}), R2.1; no longer J2.15 (P15), J2.16 (P16)
- net ~{STROBE}: now also J2.10, Q2.2 (S); no longer J2.1, RA1.3 (R3.1)
- net ~{PWREN}: now reaches U1.12 (~{PWREN})
- net ~{PWREN}: now also Q1.1 (G), R3.1
- net BUSY renamed pBUSY
- net PD0 renamed pD0
- net PD1 renamed pD1
- net PD2 renamed pD2
- net pD2: now also RA2.5 (R4.2); no longer RA3.8 (R1.2)
- net PD3 renamed pD3
- net pD3: now also RA2.6 (R3.2); no longer RA2.5 (R4.2)
- net PD4 renamed pD4
- net pD4: now also RA2.7 (R2.2); no longer RA2.6 (R3.2)
- net PD5 renamed pD5
- net pD5: now also RA2.8 (R1.2); no longer RA2.7 (R2.2)
- net PD6 renamed pD6
- net pD6: now also RA1.5 (R4.2); no longer RA2.8 (R1.2)
- net PD7 renamed pD7
- net pD7: now also RA1.6 (R3.2); no longer RA1.5 (R4.2)
- removed net ~{ACK}: J2.10, RA1.6 (R3.2)
- net ~{AUTOFD} renamed ~{pAUTOF}
- net ~{SELIN} renamed ~{pSELIN}
- net ~{pSELIN}: now also LED2.1 (K), Q2.1 (G), R5.1
- new net: LED1.1 (K), R4.1
- new net pONLINE: J2.13, J2.15 (P15), RA1.8 (R1.2)
- new net ~{pRESET}: J2.16 (P16), RA3.8 (R1.2)
- new net ~{pSTROBE}: J2.1, Q2.3 (D)
- no-connect marks 7 -> 5
Other:
- note added: "->"
- note added: "<-"
- note added: "Computer sets low to req autofeed."
- note added: "DB25 backshell snap-together 956-025-010R031 grey 956-025-010R011 black 956-025-020R121 chrome (insulate pcb!) MHCCOV-25-SN-LG grey MHCCOV-25-SN-BK black 618025214622 black"
- note added: "FDN340P"
- note added: "Printer pulses low to ack data read."
- note added: "pPE"
- note added: "~{pACK}"
- note added: "~{pERROR}"
- note removed: "Computer sets low to request auto linefeed."
- note removed: "DB25 backshell, snap-together 956-025-010R031 grey 956-025-010R011 black 956-025-020R121 chrome (insulate pcb!) MHCCOV-25-SN-LG grey MHCCOV-25-SN-BK black 618025214622 black"
- note removed: "PE"
- note removed: "Printer sets low to ack data read."
- note removed: "~{ERROR}"
- title: LPT_Capture -> LPT_Capture_DB25_MicroUSB
- moved on the sheet: C3, C4, FB1, J1, J2, RA1, U1
