File: PCB/LPT_Capture_DB25_MicroUSB_FANCY.kicad_sch (KiCad schematic)
At the start: 21 parts, among them J1 USB3155-30-A, J2 DB25P064TXLF, Q1 SL2301S, Q2 SL2301S, U1 FT245RL

Commit message: db25-microusb-fancy add R6 current limit led when /SELIN driven low
Parts:
- added R6: 10k, 000_LOCAL:R_0805, symbol 000_LOCAL:R_Small
Connections:
- net pONLINE is gone; now on net ONLINE: J2.13, J2.15 (P15), RA1.8 (R1.2)
- net ~{pSTROBE} is gone; now on net ~{STROBE}: J2.1, Q2.3 (D)
- net ONLINE: no longer LED1.2 (A), LED2.2 (A), Q1.3 (D), RA1.1 (R1.1)
- net ~{STROBE}: no longer J2.10, Q2.2 (S), R1.1, RA3.5 (R4.2)
- net pBUSY renamed BUSY
- net pD0 renamed PD0
- net pD1 renamed PD1
- net pD2 renamed PD2
- net pD3 renamed PD3
- net pD4 renamed PD4
- net pD5 renamed PD5
- net pD6 renamed PD6
- net pD7 renamed PD7
- net ~{pAUTOF} renamed ~{AUTOF}
- net ~{pRESET} renamed ~{INIT}
- net ~{pSELIN} renamed ~{SELIN}
- net ~{SELIN}: now also R6.2; no longer LED2.1 (K)
- new net: LED2.1 (K), R6.1
- new net ON: LED1.2 (A), LED2.2 (A), Q1.3 (D), RA1.1 (R1.1)
- new net ~{STR}: J2.10, Q2.2 (S), R1.1, RA3.5 (R4.2)
Other:
- note added: "PE"
- note added: "~{ACK}"
- note added: "~{ERROR}"
- note removed: "pPE"
- note removed: "~{pACK}"
- note removed: "~{pERROR}"
- moved on the sheet: R5
