File: PCB/LPT_Capture_DB25_USBC_FANCY.kicad_sch (KiCad schematic)
At the start: 21 parts, among them J1 USB3155-30-A, J2 DB25P064TXLF, Q1 SL2301S, Q2 SL2301S, U1 FT245RL

Commit message: fix db25_microusb_fancy filenames, pull db25_usbc_fancy into main
Parts:
- removed J1: USB3155-30-A, 000_LOCAL:USB3155-xx-x, symbol 000_LOCAL:USB3155-XX-X_REVA
- added J1: GSB1C4621DS2HR, 000_LOCAL:USBC_16pin_mid_mount, symbol 000_LOCAL:USBC_16pin
- added R6, R7: 5k1, 000_LOCAL:R_0805, symbol 000_LOCAL:R_Small
Connections:
- net GND: now also J1.A1B12 (GND), J1.B1A12 (GND), J1.S (SHIELD), R6.1, R7.1
- net USB+: now also J1.A6 (D+), J1.B6 (D+)
- net USB-: now also J1.A7 (D-), J1.B7 (D-)
- net VBUS: now also J1.A4B9 (VBUS), J1.B4A9 (VBUS)
- new net: J1.B5 (CC2), R7.2
- new net: J1.A5 (CC1), R6.2
- no-connect marks 5 -> 6
Other:
- note added: "DB25 LPT PRINTER INTERFACE DB25 1 ~{STROBE} - Computer pulses low when data ready. 2 PD0 ... 9 PD7 10 ~{ACK} - Printer sets low to ack data read. 11 BUSY - Printer sets high while busy. 12 PE - Printer sets high on paper end. 13 ONLINE - Printer sets high while on-line. 14 ~{AUTOFD} or Supply GND - Computer sets low to request auto linefeed, or Power GND. 15 ~{ERROR} - Printer sets low on error. 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"
- note added: "DB25 backshell, snap-together 956-025-010R031 grey 956-025-010R011 black 956-025-020R121 chrome (insulate pcb!) MHCCOV-25-SN-LG grey MHCCOV-25-SN-BK black 618025214622 black"
- note added: "USB-C Receptacle 16-pin mid-mount GSB1C4621DS2HR USB4520-03-0-A UJ20-C-H-G-MSMT-5-P16-TR"
- note removed: "->"
- note removed: "<-"
- note removed: "Computer pulses low when data ready."
- note removed: "Computer sets low to req autofeed."
- note removed: "Computer sets low to reset printer."
- note removed: "Computer sets low to select printer."
- note removed: "DB25 backshell snap-together 956-025-010R031 grey 956-025-010R011 black 956-025-020R121 chrome (insulate pcb!) MHCCOV-25-SN-LG grey MHCCOV-25-SN-BK black 618025214622 black"
- note removed: "Printer pulses low to ack data read."
- note removed: "Printer sets high on paper end."
- note removed: "Printer sets high while busy."
- note removed: "Printer sets high while on-line."
- note removed: "Printer sets low on printer error."
- title: LPT_Capture_DB25_MicroUSB_FANCY -> LPT_Capture_DB25_USBC_FANCY
- moved on the sheet: C1, C2, C3, C4, FB1, J2, LED1, LED2, N1, Q1, Q2, R1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
