File: PCB/LPT_Capture_DB25_USBC_FANCY.kicad_sch (KiCad schematic)
At the start: 23 parts, among them J1 GSB1C4621DS2HR, J2 DB25P064TXLF, Q1 SL2301S, Q2 SL2301S, U1 FT245RL

Commit message: diff pair len match
Parts:
- U1: footprint 000_LOCAL:SSOP-28_5.3x10.2mm_P0.65mm -> 000_LOCAL:SSOP-28
Changed lines of the file:
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@@
 			)
 		)
-		(property "Footprint" "000_LOCAL:SSOP-28_5.3x10.2mm_P0.65mm"
+		(property "Footprint" "000_LOCAL:SSOP-28"
 			(at 104.14 95.25 0)
 			(effects
