File: PCB/LPT_Capture_DB25_USBC_FANCY.kicad_sch (KiCad schematic)
At the start: 24 parts, among them J1 GSB1C4621DS2HR, J2 DB25P064TXLF, Q1 SL2301S, Q2 SL2301S, U1 FT245RL

Commit message: fancy versions - prevent backfeed through online led
Connections:
- net ON: no longer LED1.2 (A)
- net ONLINE: now also LED1.1 (K), R4.1; no longer RA1.8 (R1.2)
- new net: LED1.2 (A), RA1.8 (R1.2)
Other:
- moved on the sheet: LED1, LED2, R4, R5, R8
