File: PCB/LPT_Capture_Centronics_USBC_FANCY.kicad_sch (KiCad schematic)
At the start: 23 parts, among them J1 GSB1C4621DS2HR, J2 DB25P064TXLF, Q1 SL2301S, Q2 SL2301S, U1 FT245RL

Commit message: pull c36_usbc_fancy into main
Parts:
- removed J2: DB25P064TXLF, 000_LOCAL:DSUB-25_Male_EdgeMount_P2.77mm, symbol 000_LOCAL:Connector_DB25_Male
- removed N1: 956-025-010R031, 000_LOCAL:DSUB-25_Housing, symbol 000_LOCAL:Housing
- removed R3: 10k, 000_LOCAL:R_0805, symbol 000_LOCAL:R_Small
- added J2: 112-036-213R001, 000_LOCAL:Centronics_36F_RA_THT, symbol 000_LOCAL:Centronics_36
- added R1: 5K1, 000_LOCAL:R_0805, symbol 000_LOCAL:R_Small
- J1: value GSB1C4621DS2HR -> GSB1C411101DS1HR; footprint 000_LOCAL:USBC_Receptacle_16pin_mid_mount -> 000_LOCAL:USBC_Receptacle_16pin_top_mount; MPN GSB1C4621DS2HR -> GSB1C411101DS1HR
- R2: value 10k -> 5K1; MPN RC0805JR-0710KL -> RC0805FR-075K1L
- R6, R7: value 5k1 -> 10k; MPN RC0805FR-075K1L -> RC0805JR-0710KL
- U1: footprint 000_LOCAL:SSOP-28_5.3x10.2mm_P0.65mm -> 000_LOCAL:SSOP-28
- renumbered R1 to R3
Connections:
- net 3v3: now also C1.1; no longer C1.2
- net D0: now also RA3.2 (R2.1); no longer RA3.3 (R3.1)
- net D1: now also RA3.3 (R3.1); no longer RA3.2 (R2.1)
- net D2: now also RA3.4 (R4.1); no longer RA2.4 (R4.1)
- net D3: now also RA2.1 (R1.1); no longer RA2.3 (R3.1)
- net D5: now also RA2.3 (R3.1); no longer RA2.1 (R1.1)
- net D6: now also RA2.4 (R4.1); no longer RA1.4 (R4.1)
- net D7: now also RA1.1 (R1.1); no longer RA1.3 (R3.1)
- net GND: now also C1.2, R2.1, R6.2, R7.2, J2.12 (Pin_12), J2.16 (Pin_16), J2.17 (Pin_17), J2.19 (Pin_19), J2.20 (Pin_20), J2.21 (Pin_21), J2.22 (Pin_22), J2.23 (Pin_23), J2.24 (Pin_24), J2.25 (Pin_25), J2.26 (Pin_26), J2.27 (Pin_27), J2.28 (Pin_28), J2.29 (Pin_29), J2.30 (Pin_30), J2.33 (Pin_33), J2.S (Shield), R1.1; no longer C1.1, R4.2, R5.2, R6.1, R7.1
- net ONLINE: now also RA1.4 (R4.1); no longer RA1.1 (R1.1)
- net VCC: now also R4.2, R5.2, J2.35 (Pin_35); no longer R2.2
- net WR: now also Q2.2 (S), R3.1; no longer RA3.4 (R4.1)
- net pD0: now also RA3.7 (R2.2), J2.2 (Pin_2); no longer RA3.6 (R3.2)
- net pD1: now also RA3.6 (R3.2), J2.3 (Pin_3); no longer RA3.7 (R2.2)
- net pD2: now also RA3.5 (R4.2), J2.4 (Pin_4); no longer RA2.5 (R4.2)
- net pD3: now also RA2.8 (R1.2), J2.5 (Pin_5); no longer RA2.6 (R3.2)
- net pD4: now also J2.6 (Pin_6)
- net pD5: now also RA2.6 (R3.2), J2.7 (Pin_7); no longer RA2.8 (R1.2)
- net pD6: now also RA2.5 (R4.2), J2.8 (Pin_8); no longer RA1.5 (R4.2)
- net pD7: now also RA1.8 (R1.2), J2.9 (Pin_9); no longer RA1.6 (R3.2)
- net pONLINE: now also RA1.5 (R4.2), J2.13 (Pin_13), J2.18 (Pin_18), J2.32 (Pin_32); no longer RA1.8 (R1.2)
- net ~{PWREN}: now also R5.1
- net ~{RESET}: now also R4.1, RA1.3 (R3.1); no longer R2.1, RA3.1 (R1.1)
- net ~{STROBE}: now also Q2.3 (D), RA3.1 (R1.1); no longer Q2.2 (S), R3.1, RA3.5 (R4.2)
- net ~{pRESET}: now also RA1.6 (R3.2), J2.31 (Pin_31); no longer RA3.8 (R1.2)
- net ~{pSTROBE}: now also RA3.8 (R1.2), J2.1 (Pin_1), J2.10 (Pin_10); no longer Q2.3 (D)
- net at LED1.1 (K): now also R6.1; no longer R4.1
- net at J1.B5 (CC2): now also R2.2; no longer R7.2
- net at J1.A5 (CC1): now also R1.2; no longer R6.2
- net pBUSY renamed BUSY
- net BUSY: now also J2.11 (Pin_11)
- net ~{pSELIN} renamed ~{SELIN}
- net ~{SELIN}: now also R7.1, J2.36 (Pin_36); no longer R5.1
- new net ~{AUTOFD}: J2.14 (Pin_14)
- no-connect marks 6 -> 8
Other:
- note added: "->"
- note added: "5V"
- note added: "<-"
- note added: "CENTRONICS PRINTER INTERFACE 1 ~{STROBE} - Computer pulses low when data ready. 2 PD0 ... 9 PD7 10 ~{ACK} - Printer sets low to ack data read. 11 BUSY - Printer sets high while busy. 12 PE - Printer sets high on paper end. 13 ONLINE - Printer sets high while on-line. 14 ~{AUTOFD} or Supply GND - Computer sets low to request auto linefeed, or Power GND. 15 OSCTX - Oscillator Transmit, 100-200 KHz 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"
- note added: "Centronics 36 Female FUY57005 FUY57010 FUY57075 112-036-213R001 112-036-213R491 1734044-1 1734044-2 1734044-3 5552742-1 5555119-1 5555233-1"
- note added: "Chassis GND"
- note added: "GND"
- note added: "OSCTX"
- note added: "PE"
- note added: "PLH"
- note added: "Signal GND"
- note added: "USB-C Receptacle, 16-pin, top-mount UJ20-C-H-G-SMT-P16-TR GSB1C411101DS1HR USB4105-GF-A-120"
- note added: "~{ACK}"
- note added: "~{ERROR}"
- note removed: "DB25 LPT PRINTER INTERFACE DB25 1 ~{STROBE} - Computer pulses low when data ready. 2 PD0 ... 9 PD7 10 ~{ACK} - Printer sets low to ack data read. 11 BUSY - Printer sets high while busy. 12 PE - Printer sets high on paper end. 13 ONLINE - Printer sets high while on-line. 14 ~{AUTOFD} or Supply GND - Computer sets low to request auto linefeed, or Power GND. 15 ~{ERROR} - Printer sets low on error. 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"
- note removed: "DB25 Male solder-cup Fits 1.6mm PCB: DB25P064TXLF A-DS 25 LL/Z - loose DE25PNES - tight, slide in from side L717SDB25P 61802524823 2101-0180-03 Needs 1.2mm PCB: 171-025-103L001 MHDB25SP DB25-PD 40-9725M"
- note removed: "DB25 backshell, snap-together 956-025-010R031 grey 956-025-010R011 black 956-025-020R121 chrome (insulate pcb!) MHCCOV-25-SN-LG grey MHCCOV-25-SN-BK black 618025214622 black"
- note removed: "FDN340P"
- note removed: "USB-C Receptacle 16-pin mid-mount GSB1C4621DS2HR USB4520-03-0-A UJ20-C-H-G-MSMT-5-P16-TR"
- note removed: "pPE"
- note removed: "~{pACK}"
- note removed: "~{pERROR}"
- title: LPT_Capture_DB25_USBC_FANCY -> LPT_Capture_C36_USBC
- moved on the sheet: C2, C3, C4, FB1, LED1, LED2, Q1, Q2, R3, RA1, U1
