File: PCB/LPT_Capture_Centronics_USBC_FANCY.kicad_sch (KiCad schematic)
At the start: 22 parts, among them J1 GSB1C411101DS1HR, J2 112-036-213R001, Q1 SL2301S, Q2 SL2301S, U1 FT245RL

Commit message: centronics control flow arrows
Other:
- note removed: "->"
- note removed: "<-"
