File: PCB/LPT_Capture_DB25_USBC_BASIC.kicad_sch (KiCad schematic)
At the start: 15 parts, among them J1 GSB1C4621DS2HR, J2 DB25P064TXLF, U1 FT245RL

Commit message: pull c36_usbc_fancy into main
Parts:
- J1: footprint 000_LOCAL:USBC_16pin_mid_mount -> 000_LOCAL:USBC_Receptacle_16pin_mid_mount
Changed lines of the file:
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@@
 			)
 		)
-		(property "Footprint" "000_LOCAL:USBC_16pin_mid_mount"
+		(property "Footprint" "000_LOCAL:USBC_Receptacle_16pin_mid_mount"
 			(at 49.53 88.9 0)
 			(effects
