File: PCB/LPT_Capture_CN36_USBC_FANCY.kicad_sch (KiCad schematic)
At the start: 26 parts, among them J1 GSB1C411101DS1HR, J2 112-036-213R001, Q1 SL2301S, Q2 SL2301S, SW1 SW_DIP_x04, U1 FT245RL

Commit message: cn36 add jp1,2,3
Parts:
- added JP1: GND_USBSHLD, 000_LOCAL:SolderJumper-2_P1.3mm_Bridged_RoundedPad1.0x1.5mm, symbol 000_LOCAL:Jumper_2_Small_Bridged
- added JP2: GND_LPTSHLD, 000_LOCAL:SolderJumper-2_P1.3mm_Bridged_RoundedPad1.0x1.5mm, symbol 000_LOCAL:Jumper_2_Small_Bridged
- added JP3: USBSHLD_LPTSHLD, 000_LOCAL:SolderJumper-2_P1.3mm_Bridged_RoundedPad1.0x1.5mm, symbol 000_LOCAL:Jumper_2_Small_Bridged
Connections:
- net GND: now also JP1.1 (A), JP2.1 (A); no longer J1.S (SHIELD), J2.17 (Pin_17), J2.S (Shield)
- new net LPT_SHIELD: J2.17 (Pin_17), J2.S (Shield), JP2.2 (B), JP3.2 (B)
- new net USB_SHIELD: J1.S (SHIELD), JP1.2 (B), JP3.1 (A)
Other:
- note added: "(1%)"
