File: PCB/LPT_Capture_CN36_USBC_FANCY.kicad_sch (KiCad schematic)
At the start: 30 parts, among them J1 GSB1C411101DS1HR, J2 112-036-213R001, Q1 SL2301S, Q2 SL2301S, SW1 SW_DIP_x04, U1 FT245RL

Commit message: fancy versions - prevent backfeed through online led
Connections:
- net ON: now also LED1.1 (K), R6.1; no longer LED1.2 (A), LED2.2 (A), Q1.3 (D)
- new net: LED1.2 (A), LED2.2 (A), Q1.3 (D)
Other:
- moved on the sheet: LED1, LED2, R6, R8
Changed lines of the file:
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@@
 	(title_block
 		(title "LPT_Capture_CN36_USBC_FANCY")
-		(date "2025-12-24")
-		(rev "006")
+		(date "2026-03-25")
+		(rev "007")
 		(company "b.kenyon.w@gmail.com")
 		(comment 1 "CC-BY-SA")
@@
 	)
 	(junction
+		(at 180.34 106.68)
+		(diameter 0)
+		(color 0 0 0 0)
+	)
+	(junction
+		(at 158.75 106.68)
+		(diameter 0)
+		(color 0 0 0 0)
+	)
+	(junction
 		(at 226.06 106.68)
 		(diameter 0)
@@
 	)
 	(junction
-		(at 88.9 38.1)
+		(at 170.18 106.68)
 		(diameter 0)
 		(color 0 0 0 0)
 	)
 	(junction
-		(at 138.43 106.68)
+		(at 88.9 38.1)
 		(diameter 0)
 		(color 0 0 0 0)
 	)
 	(junction
-		(at 50.8 78.74)
+		(at 138.43 106.68)
 		(diameter 0)
 		(color 0 0 0 0)
 	)
 	(junction
-		(at 76.2 104.14)
+		(at 50.8 78.74)
 		(diameter 0)
 		(color 0 0 0 0)
 	)
 	(junction
-		(at 152.4 106.68)
+		(at 76.2 104.14)
 		(diameter 0)
 		(color 0 0 0 0)
@@
 	)
 	(junction
-		(at 165.1 106.68)
-		(diameter 0)
-		(color 0 0 0 0)
-	)
-	(junction
 		(at 248.92 118.11)
 		(diameter 0)
@@
 	)
 	(junction
-		(at 180.34 106.68)
-		(diameter 0)
-		(color 0 0 0 0)
-	)
-	(junction
 		(at 101.6 119.38)
 		(diameter 0)
@@
 	(wire
 		(pts
-			(xy 152.4 106.68) (xy 165.1 106.68)
-		)
-		(stroke
-			(width 0)
-			(type default)
-		)
-	)
-	(wire
-		(pts
 			(xy 212.09 109.22) (xy 223.52 109.22)
 		)
@@
 		)
 	)
-	(wire
-		(pts
-			(xy 165.1 106.68) (xy 180.34 106.68)
-		)
-		(stroke
-			(width 0)
-			(type default)
-		)
-	)
 	(polyline
 		(pts
@@
 	(wire
 		(pts
-			(xy 165.1 119.38) (xy 175.26 119.38)
+			(xy 158.75 119.38) (xy 175.26 119.38)
 		)
 		(stroke
@@
 	(wire
 		(pts
-			(xy 148.59 106.68) (xy 152.4 106.68)
+			(xy 148.59 106.68) (xy 158.75 106.68)
+		)
+		(stroke
+			(width 0)
+			(type default)
+		)
+	)
+	(wire
+		(pts
+			(xy 170.18 106.68) (xy 170.18 109.22)
 		)
 		(stroke
@@
 	(wire
 		(pts
+			(xy 170.18 106.68) (xy 180.34 106.68)
+		)
+		(stroke
+			(width 0)
+			(type default)
+		)
+	)
+	(wire
+		(pts
 			(xy 260.35 104.14) (xy 256.54 104.14)
 		)
@@
 		)
 	)
+	(wire
+		(pts
+			(xy 158.75 106.68) (xy 162.56 106.68)
+		)
+		(stroke
+			(width 0)
+			(type default)
+		)
+	)
 	(polyline
 		(pts
@@
 		)
 	)
-	(label "ON"
-		(at 148.59 106.68 0)
-		(effects
-			(font
-				(size 1.27 1.27)
-			)
-			(justify left bottom)
-		)
-	)
 	(label "PD1"
 		(at 208.28 73.66 0)
@@
 	(symbol
 		(lib_id "000_LOCAL:R_Small")
-		(at 165.1 116.84 0)
+		(at 158.75 116.84 0)
 		(mirror y)
 		(unit 1)
@@
 		(dnp no)
 		(property "Reference" "R8"
-			(at 166.624 115.824 0)
+			(at 160.274 115.824 0)
 			(effects
 				(font
@@
 		)
 		(property "Value" "10k"
-			(at 166.624 117.856 0)
+			(at 160.274 117.856 0)
 			(effects
 				(font
@@
 		)
 		(property "Footprint" "000_LOCAL:R_0805"
-			(at 165.1 116.84 0)
+			(at 158.75 116.84 0)
 			(effects
 				(font
@@
 		)
 		(property "Datasheet" "datasheets/PYU-RC_GROUP_51_ROHS_L.pdf"
-			(at 165.1 116.84 0)
+			(at 158.75 116.84 0)
 			(effects
 				(font
@@
 		)
 		(property "Description" "RES 10K OHM 5% 1/8W 0805"
-			(at 165.1 116.84 0)
+			(at 158.75 116.84 0)
 			(effects
 				(font
@@
 		)
 		(property "MPN" "RC0805JR-0710KL"
-			(at 165.1 116.84 0)
+			(at 158.75 116.84 0)
 			(effects
 				(font
@@
 	(symbol
 		(lib_id "000_LOCAL:R_Small")
-		(at 152.4 116.84 0)
+		(at 170.18 111.76 0)
 		(mirror y)
 		(unit 1)
@@
 		(dnp no)
 		(property "Reference" "R6"
-			(at 154.178 116.586 0)
+			(at 171.958 111.506 0)
 			(effects
 				(font
@@
 		)
 		(property "Value" "10k"
-			(at 154.178 118.872 0)
+			(at 171.958 113.792 0)
 			(effects
 				(font
@@
 		)
 		(property "Footprint" "000_LOCAL:R_0805"
-			(at 152.4 116.84 0)
+			(at 170.18 111.76 0)
 			(effects
 				(font
@@
 		)
 		(property "Datasheet" "datasheets/PYU-RC_GROUP_51_ROHS_L.pdf"
-			(at 152.4 116.84 0)
+			(at 170.18 111.76 0)
 			(effects
 				(font
@@
 		)
 		(property "Description" "RES 10K OHM 5% 1/8W 0805"
-			(at 152.4 116.84 0)
+			(at 170.18 111.76 0)
 			(effects
 				(font
@@
 		)
 		(property "MPN" "RC0805JR-0710KL"
-			(at 152.4 116.84 0)
+			(at 170.18 111.76 0)
 			(effects
 				(font
@@
 	(symbol
 		(lib_id "000_LOCAL:LED")
-		(at 165.1 110.49 90)
+		(at 158.75 110.49 90)
 		(unit 1)
 		(exclude_from_sim no)
@@
 		(dnp no)
 		(property "Reference" "LED2"
-			(at 167.64 109.22 90)
+			(at 158.75 102.362 90)
 			(effects
 				(font
 					(size 1.27 1.27)
 				)
-				(justify right)
 			)
 		)
 		(property "Value" "LTL-307GLC"
-			(at 160.02 116.332 90)
+			(at 153.67 116.332 90)
 			(effects
 				(font
@@
 		)
 		(property "Footprint" "000_LOCAL:LED_D5.0mm"
-			(at 165.1 110.49 0)
+			(at 158.75 110.49 0)
 			(effects
 				(font
@@
 		)
 		(property "Datasheet" "datasheets/LTL-307GLC.pdf"
-			(at 165.1 110.49 0)
+			(at 158.75 110.49 0)
 			(effects
 				(font
@@
 		)
 		(property "Description" "Light emitting diode"
-			(at 165.1 110.49 0)
+			(at 158.75 110.49 0)
 			(effects
 				(font
@@
 		)
 		(property "Sim.Pins" "1=K 2=A"
-			(at 165.1 110.49 0)
+			(at 158.75 110.49 0)
 			(effects
 				(font
@@
 		)
 		(property "MPN" "LTL-307GLC"
-			(at 165.1 110.49 90)
+			(at 158.75 110.49 90)
 			(effects
 				(font
@@
 		)
 		(property "LABEL" "SELECT"
-			(at 170.942 111.506 90)
+			(at 158.75 104.648 90)
 			(effects
 				(font
@@
 	(symbol
 		(lib_id "000_LOCAL:LED")
-		(at 152.4 110.49 90)
+		(at 166.37 106.68 180)
 		(unit 1)
 		(exclude_from_sim no)
@@
 		(dnp no)
 		(property "Reference" "LED1"
-			(at 154.94 109.22 90)
+			(at 166.37 100.838 0)
 			(effects
 				(font
 					(size 1.27 1.27)
 				)
-				(justify right)
 			)
 		)
 		(property "Value" "LTL-307GLC"
-			(at 150.876 113.284 90)
+			(at 169.164 108.204 90)
 			(effects
 				(font
@@
 		)
 		(property "Footprint" "000_LOCAL:LED_D5.0mm"
-			(at 152.4 110.49 0)
+			(at 166.37 106.68 0)
 			(effects
 				(font
@@
 		)
 		(property "Datasheet" "datasheets/LTL-307GLC.pdf"
-			(at 152.4 110.49 0)
+			(at 166.37 106.68 0)
 			(effects
 				(font
@@
 		)
 		(property "Description" "Light emitting diode"
-			(at 152.4 110.49 0)
+			(at 166.37 106.68 0)
 			(effects
 				(font
@@
 		)
 		(property "Sim.Pins" "1=K 2=A"
-			(at 152.4 110.49 0)
+			(at 166.37 106.68 0)
 			(effects
 				(font
@@
 		)
 		(property "MPN" "LTL-307GLC"
-			(at 152.4 110.49 90)
+			(at 166.37 106.68 90)
 			(effects
 				(font
@@
 		)
 		(property "LABEL" "ONLINE"
-			(at 158.242 111.506 90)
+			(at 166.37 102.87 0)
 			(effects
 				(font
@@
 	(symbol
 		(lib_id "power:GND")
-		(at 152.4 119.38 0)
+		(at 170.18 114.3 0)
 		(unit 1)
 		(exclude_from_sim no)
@@
 		(dnp no)
 		(property "Reference" "#PWR017"
-			(at 152.4 125.73 0)
+			(at 170.18 120.65 0)
 			(effects
 				(font
@@
 		)
 		(property "Value" "GND"
-			(at 152.654 124.206 0)
+			(at 170.434 119.126 0)
 			(effects
 				(font
@@
 		)
 		(property "Footprint" ""
-			(at 152.4 119.38 0)
+			(at 170.18 114.3 0)
 			(effects
 				(font
@@
 		)
 		(property "Datasheet" ""
-			(at 152.4 119.38 0)
+			(at 170.18 114.3 0)
 			(effects
 				(font
@@
 		)
 		(property "Description" ""
-			(at 152.4 119.38 0)
+			(at 170.18 114.3 0)
 			(effects
 				(font
