File: PCB/LPT_Capture_CN36_USBC_FANCY.kicad_sch (KiCad schematic)
At the start: 30 parts, among them J1 GSB1C411101DS1HR, J2 112-036-213R001, Q1 SL2301S, Q2 SL2301S, SW1 SW_DIP_x04, U1 FT245RL

Commit message: cn36 add reset button
Parts:
- added SW2: RESET, 000_LOCAL:SW_SPST_PTS810, symbol 000_LOCAL:SW_Push
Connections:
- net GND: now also SW2.1
- net PLH: now also RA4.5 (R4.2); no longer RA4.6 (R3.2)
- net sPLH: now also RA4.4 (R4.1); no longer RA4.3 (R3.1)
- net ~{RESET}: now also SW2.2
- net ~{SELIN}: now also RA4.6 (R3.2); no longer RA4.5 (R4.2)
- net ~{SEL}: now also RA4.3 (R3.1); no longer RA4.4 (R4.1)
- net PWREN: now reaches LED1.2 (A), LED2.2 (A), Q1.3 (D)
- net sERR renamed ~{sERR}
Other:
- moved on the sheet: LED1, LED2, R6, R8
